File: NotSoLite-S3/NotSoLite-S3.kicad_pcb (KiCad board)
At the start: 4 copper layers, 25 x 50 mm, 46 parts, among them J1 USB_C_Receptacle_USB2.0_16P, J2 Battery_Pad, J3 Conn_01x13, J4 Conn_01x13, SW1 SW_Push, SW2 SW_Push, U1 ESP32-S3, U2 ZD25WQ32CEIGR, U3 MIC5205-3.3YM5, U4 TP4057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

Commit message: fucked BB converter attempt
Parts:
- added D5: EMERALD, LED_SMD:LED_0402_1005Metric, F.Cu at (108.4, 80.2)
- added G***: LOGO, LOGO, F.Cu at (111.7, 77.8)
- added G***: LOGO, LOGO, B.Cu at (107.3, 70.8)
- added G***: LOGO, LOGO, B.Cu at (117.3, 70.9)
- added G***: LOGO, LOGO, B.Cu at (112.0, 85.9)
- added G***: LOGO, LOGO, B.Cu at (117.1, 80.7)
- added G***: LOGO, LOGO, B.Cu at (117.0, 76.5)
- added G***: LOGO, LOGO, B.Cu at (117.0, 78.5)
- added G***: LOGO, LOGO, B.Cu at (110.7, 61.7)
- added G***: LOGO, LOGO, B.Cu at (116.9, 62.5)
- added R11: 330, Resistor_SMD:R_0402_1005Metric, F.Cu at (108.4, 78.2)
- moved R4 97.7 mm to (120.8, 90.6), turned to 90 degrees
- moved R3 96.8 mm to (117.8, 90.6), turned to 90 degrees
- moved D1 94.8 mm to (115.5, 87.6), turned to -90 degrees
- moved C13 94.4 mm to (113.5, 91.2)
- moved R1 93.4 mm to (111.9, 92.8)
- moved R5 93.3 mm to (118.7, 88.2), turned to 90 degrees
- moved R6 93.0 mm to (119.8, 88.2), turned to 90 degrees
- moved U2 92.6 mm to (112.0, 73.1), turned to 180 degrees
- moved C3 89.5 mm to (118.7, 60.9)
- moved C17 89.1 mm to (118.8, 79.6)
- moved C5 88.9 mm to (118.7, 61.9)
- moved C10 87.5 mm to (118.2, 67.4)
- moved R8 87.3 mm to (113.1, 86.7)
- moved C16 86.9 mm to (120.3, 67.6), turned to 180 degrees
- moved C18 86.6 mm to (115.7, 78.9), turned to 180 degrees
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Connections:
- J4 pad 1: VBUS -> +3V3
- J4 pad 2: +3V3 -> VBUS
Routing:
- net /RESET: track 0.89 -> 53.5 mm, vias 1 -> 2
- net /USB_DM: track 0.00 -> 40.5 mm
- net /USB_DP: track 0.00 -> 39.5 mm
- net /P10: track 0.00 -> 39.1 mm, vias 0 -> 1
- net /P11: track 0.00 -> 36.3 mm, vias 0 -> 1
- net /P12: track 0.00 -> 34.0 mm, vias 0 -> 1
- net /P18: track 0.00 -> 33.4 mm, vias 0 -> 1
- net /P13: track 0.00 -> 32.8 mm, vias 0 -> 1
- net /P14: track 0.00 -> 31.3 mm, vias 0 -> 1
- net /P17: track 0.00 -> 31.2 mm, vias 0 -> 1
- net /BOOT: track 1.12 -> 20.7 mm, vias 1 -> 2
- net /FLASH_CLK: track 0.00 -> 12.1 mm, vias 0 -> 2
- net /FLASH_D1: track 0.00 -> 11.1 mm
- net /P21: track 0.00 -> 10.4 mm, vias 0 -> 2
- net /FLASH_D0: track 0.00 -> 8.43 mm, vias 0 -> 2
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- added copper zone on F.Cu, net +3V3
- added copper zone on In2.Cu, net +3V3
- added copper zone on In3.Cu, net GND
- added copper zone on In4.Cu, net GND
- added copper zone on F.Cu, net Net-(J2-Pin_1)
- added copper zone on F.Cu, net SPIPWR
- added copper zone on In2.Cu, net SPIPWR
- added copper zone on F.Cu, net VBUS
- added copper zone on In2.Cu, net VBUS
- added copper zone on F.Cu, net VSYS
Other:
- copper layers 4 -> 6
- board text added: "+3V3"
- board text added: "94V-0 E479892 JLC-1"
- board text added: "@mastodon.social"
- board text added: "@zeankun.dev"
- board text added: "BOOT"
- board text added: "C"
- board text added: "FROM THE RIVER TO THE SEA, PALESTINE WILL BE FREE!"
- board text added: "GND"
- board text added: "LIPO IN LI-ION IN"
- board text added: "P1"
- board text added: "P10"
- board text added: "P11"
- board text added: "P12"
- board text added: "P13"
- board text added: "P14"
- board text added: "P17"
- board text added: "P18"
- board text added: "P2"
- board text added: "P3"
- board text added: "P4"
- board text added: "P5"
- board text added: "P6"
- board text added: "P7"
- board text added: "P8"
- board text added: "P9"
- board text added: "RESET"
- board text added: "US"
- board text added: "VBUS"
- board text added: "by purchasing any zeankun.dev product, you are helping people in palestine. thank you so much for your kindness :)"
- board text added: "designed on a workstation by:"
- board text added: "love it? i'd like to hear from you!"
- board text added: "zeankun.dev's NotSoLite ESP32-S3"
- board text added: "zeankundev"
- board text added: "©️ 2024 zeankun.dev. logo ©️ choco panda kat all rights reserved"
