File: NotSoLite-S3/NotSoLite-S3.kicad_sch (KiCad schematic)
At the start: 46 parts, among them J1 USB_C_Receptacle_USB2.0_16P, J2 Battery_Pad, J3 Conn_01x13, J4 Conn_01x13, SW1 SW_Push, SW2 SW_Push, U1 ESP32-S3, U2 ZD25WQ32CEIGR, U3 MIC5205-3.3YM5, U4 TP4057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

Commit message: fucked BB converter attempt
Parts:
- added D5: EMERALD, LED_SMD:LED_0402_1005Metric, symbol Device:LED
- added R11: 330, Resistor_SMD:R_0402_1005Metric, symbol Device:R
Connections:
- net +3V3: now also J4.1 (Pin_1); no longer J4.2 (Pin_2)
- net GND: now also D5.1 (K)
- net P21: now also R11.1
- net VBUS: now also J4.2 (Pin_2); no longer J4.1 (Pin_1)
- new net: D5.2 (A), R11.2
Other:
- moved on the sheet: C15, C16, Y1
