File: CastleBox/CastleBox.kicad_pcb (KiCad board)
At the start: 6 copper layers, 50 x 33 mm, 43 parts, among them J1 USB_C_Receptacle_USB2.0_16P, J2 HDMI_C_1.4, J4 Conn_02x15_Odd_Even, U1 XC6SLX9-FTG256, U2 MIC5205YM5, U3 MIC5205YM5, U4 W955K8MBYA, U5 W955K8MBYA, U6 CY7C65215-32LTXI, X1 ASE-50MHz

Commit message: routine backup
Parts:
- added C19: 0.1u, Capacitor_SMD:C_0402_1005Metric, F.Cu at (86.7, 67.6)
- added C20: 0.1u, Capacitor_SMD:C_0402_1005Metric, F.Cu at (79.6, 64.7)
- added G***: LOGO, LOGO, B.Cu at (100.6, 76.4)
- added G***: LOGO, LOGO, B.Cu at (102.8, 63.9)
- added G***: LOGO, LOGO, B.Cu at (93.2, 76.3)
- added G***: LOGO, LOGO, B.Cu at (93.2, 72.1)
- added G***: LOGO, LOGO, B.Cu at (93.2, 74.1)
- added G***: LOGO, LOGO, B.Cu at (95.2, 68.0)
- added G***: LOGO, LOGO, B.Cu at (95.6, 84.8)
- added G***: LOGO, LOGO, B.Cu at (110.8, 78.9)
- added R11: 100k, Resistor_SMD:R_0402_1005Metric, F.Cu at (73.8, 63.4)
- added R12: 100k, Resistor_SMD:R_0402_1005Metric, F.Cu at (73.8, 62.4)
- added REF**: KiCad-Logo2_5mm_SilkScreen, Symbol:KiCad-Logo2_5mm_SilkScreen, B.Cu at (83.9, 85.7)
- added U7: TXS0102YZP, Package_BGA:Texas_DSBGA-8_0.9x1.9mm_Layout2x4_P0.5mm, F.Cu at (83.0, 67.2)
- J2: footprint Connector_Video:HDMI_Micro-D_Molex_46765-1x01 -> HDMI:VALCON_HD-RA-DSF12-TR
- moved U2 62.0 mm to (81.8, 87.0)
- moved R2 54.6 mm to (85.8, 87.6), turned to 90 degrees
- moved R1 54.6 mm to (84.6, 86.6), turned to 90 degrees
- moved C2 51.0 mm to (87.7, 88.1)
- moved C1 50.3 mm to (88.2, 84.8)
- moved C18 50.2 mm to (84.7, 78.6), turned to -90 degrees
- moved R4 49.5 mm to (85.9, 84.2), turned to -90 degrees
- moved R3 49.4 mm to (84.9, 83.2), turned to -90 degrees
- moved C3 48.1 mm to (87.2, 86.6), turned to -90 degrees
- moved C4 44.1 mm to (87.3, 83.2), turned to -90 degrees
- moved U3 43.2 mm to (81.8, 83.6)
- moved R6 40.5 mm to (78.3, 83.1), turned to -90 degrees
- moved D1 40.2 mm to (76.6, 88.0), turned to 180 degrees
- moved R5 39.5 mm to (79.0, 78.8)
- moved R9 35.8 mm to (86.6, 76.1), turned to 90 degrees
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Connections:
- J2 pad 1: unconnected-(J2-D2S-Pad1) -> GND
- J2 pad 10: unconnected-(J2-CKS-Pad10) -> GND
- J2 pad 13: unconnected-(J2-GND-Pad13) -> GND
- J2 pad 15: unconnected-(J2-SCL-Pad15) -> Net-(J2-SCL)
- J2 pad 16: unconnected-(J2-SDA-Pad16) -> Net-(J2-SDA)
- J2 pad 18: unconnected-(J2-+5V-Pad18) -> VSYS
- J2 pad 19: unconnected-(J2-HPD/HEAC--Pad19) -> Net-(J2-HPD/HEAC-)
- J2 pad 4: unconnected-(J2-D1S-Pad4) -> GND
- J2 pad 7: unconnected-(J2-D0S-Pad7) -> GND
- J2 pad SH: unconnected-(J2-PadSH) -> GND
- J4 pad 1: unconnected-(J4-Pin_1-Pad1) -> VBUS
- J4 pad 10: unconnected-(J4-Pin_10-Pad10) -> /PA4
- J4 pad 11: unconnected-(J4-Pin_11-Pad11) -> /PA6
- J4 pad 12: unconnected-(J4-Pin_12-Pad12) -> /PB5
- J4 pad 13: unconnected-(J4-Pin_13-Pad13) -> /PA7
- J4 pad 14: unconnected-(J4-Pin_14-Pad14) -> /PB6
- J4 pad 15: unconnected-(J4-Pin_15-Pad15) -> /PA8
- J4 pad 16: unconnected-(J4-Pin_16-Pad16) -> /PB8
- J4 pad 17: unconnected-(J4-Pin_17-Pad17) -> /PB10
- J4 pad 18: unconnected-(J4-Pin_18-Pad18) -> /PA9
- J4 pad 19: unconnected-(J4-Pin_19-Pad19) -> /PA11
- J4 pad 2: unconnected-(J4-Pin_2-Pad2) -> +1V2
- J4 pad 20: unconnected-(J4-Pin_20-Pad20) -> /PA12
- J4 pad 21: unconnected-(J4-Pin_21-Pad21) -> /PB12
- J4 pad 22: unconnected-(J4-Pin_22-Pad22) -> GND
- J4 pad 23: unconnected-(J4-Pin_23-Pad23) -> /PB14
- J4 pad 24: unconnected-(J4-Pin_24-Pad24) -> /PA13
- J4 pad 25: unconnected-(J4-Pin_25-Pad25) -> /PB15
- J4 pad 26: unconnected-(J4-Pin_26-Pad26) -> /PA14
- J4 pad 27: unconnected-(J4-Pin_27-Pad27) -> +3V3
- J4 pad 29: unconnected-(J4-Pin_29-Pad29) -> VSYS
- J4 pad 3: unconnected-(J4-Pin_3-Pad3) -> /PA2
- J4 pad 30: unconnected-(J4-Pin_30-Pad30) -> GND
- J4 pad 4: unconnected-(J4-Pin_4-Pad4) -> GND
- J4 pad 5: unconnected-(J4-Pin_5-Pad5) -> /PC3
- J4 pad 6: unconnected-(J4-Pin_6-Pad6) -> /PC2
- J4 pad 7: unconnected-(J4-Pin_7-Pad7) -> /PB3
- J4 pad 8: unconnected-(J4-Pin_8-Pad8) -> /PA3
- J4 pad 9: unconnected-(J4-Pin_9-Pad9) -> /PA5
- U1 pad A11: unconnected-(U1A-IO_L39N_0-PadA11) -> /PA11
- U1 pad A12: unconnected-(U1A-IO_L62N_VREF_0-PadA12) -> /PA12
- U1 pad A13: unconnected-(U1A-IO_L63N_SCP6_0-PadA13) -> /PA13
- U1 pad A14: unconnected-(U1A-IO_L65N_SCP2_0-PadA14) -> /PA14
- U1 pad A2: unconnected-(U1B-IO_L52N_M3A9_3-PadA2) -> /PA2
- U1 pad A3: unconnected-(U1B-IO_L83N_VREF_3-PadA3) -> /PA3
- U1 pad A4: unconnected-(U1A-IO_L1N_VREF_0-PadA4) -> /PA4
- U1 pad A5: unconnected-(U1A-IO_L2N_0-PadA5) -> /PA5
- U1 pad A6: unconnected-(U1A-IO_L4N_0-PadA6) -> /PA6
- U1 pad A7: unconnected-(U1A-IO_L6N_0-PadA7) -> /PA7
- U1 pad A8: unconnected-(U1A-IO_L33N_0-PadA8) -> /PA8
- U1 pad A9: unconnected-(U1A-IO_L34N_GCLK18_0-PadA9) -> /PA9
- U1 pad B1: unconnected-(U1B-IO_L50N_M3BA2_3-PadB1) -> /CK+
- U1 pad B10: unconnected-(U1A-IO_L35P_GCLK17_0-PadB10) -> /PB10
- U1 pad B12: unconnected-(U1A-IO_L62P_0-PadB12) -> /PB12
- U1 pad B14: unconnected-(U1A-IO_L65P_SCP3_0-PadB14) -> /PB14
- U1 pad B15: unconnected-(U1A-IO_L29P_A23_M1A13_1-PadB15) -> /PB15
- U1 pad B2: unconnected-(U1B-IO_L52P_M3A8_3-PadB2) -> /CK-
- U1 pad B3: unconnected-(U1B-IO_L83P_3-PadB3) -> /PB3
- U1 pad B5: unconnected-(U1A-IO_L2P_0-PadB5) -> /PB5
- U1 pad B6: unconnected-(U1A-IO_L4P_0-PadB6) -> /PB6
- U1 pad B8: unconnected-(U1A-IO_L33P_0-PadB8) -> /PB8
- U1 pad C1: unconnected-(U1B-IO_L50P_M3WE_3-PadC1) -> /D0+
- U1 pad C2: unconnected-(U1B-IO_L48N_M3BA1_3-PadC2) -> /PC2
- U1 pad C3: unconnected-(U1B-IO_L48P_M3BA0_3-PadC3) -> /PC3
- U1 pad D1: unconnected-(U1B-IO_L49N_M3A2_3-PadD1) -> /D0-
- U1 pad D3: unconnected-(U1B-IO_L49P_M3A7_3-PadD3) -> /DVI_SCL
- U1 pad E1: unconnected-(U1B-IO_L46N_M3CLKN_3-PadE1) -> /D1+
- U1 pad E2: unconnected-(U1B-IO_L46P_M3CLK_3-PadE2) -> /D1-
- U1 pad E3: unconnected-(U1B-IO_L54N_M3A11_3-PadE3) -> /DVI_SDA
- U1 pad F1: unconnected-(U1B-IO_L41N_GCLK26_M3DQ5_3-PadF1) -> /D2-
- U1 pad F2: unconnected-(U1B-IO_L41P_GCLK27_M3DQ4_3-PadF2) -> /DVI_HOTPLUG
- U1 pad G1: unconnected-(U1B-IO_L40N_M3DQ7_3-PadG1) -> /D2+
Routing:
- net /FPGA_TDO: track 0.00 -> 36.5 mm, vias 0 -> 2
- net /FPGA_TCK: track 0.00 -> 32.3 mm, vias 0 -> 2
- net /FPGA_TMS: track 0.00 -> 30.7 mm, vias 0 -> 2
- net /FPGA_TDI: track 0.00 -> 30.6 mm, vias 0 -> 2
- net /D1+: track 0.00 -> 26.0 mm
- net /D1-: track 0.00 -> 25.9 mm, vias 0 -> 2
- net /DVI_HOTPLUG: track 0.00 -> 25.3 mm, vias 0 -> 2
- net GND: track 37.3 -> 59.4 mm, vias 41 -> 76
- net /PC2: track 0.00 -> 21.5 mm
- net /CK+: track 0.00 -> 19.3 mm
- net /D0-: track 0.00 -> 18.2 mm
- net /D0+: track 0.00 -> 18.2 mm, vias 0 -> 1
- net /CK-: track 0.00 -> 18.0 mm, vias 0 -> 1
- net /D2+: track 0.00 -> 17.9 mm
- net /PC3: track 0.00 -> 17.8 mm
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- added copper zone on F.Cu, net +1V2
- added copper zone on In2.Cu, net +1V2
- added copper zone on F.Cu, net +3V3
- added copper zone on In4.Cu, net GND
- added copper zone on F.Cu, net VBUS
- added copper zone on In3.Cu, net VBUS
- added copper zone on F.Cu, net VSYS
- added copper zone on In3.Cu, net VSYS
- removed copper zone on In4.Cu, net +1V2
- removed copper zone on In2.Cu, net GND
- removed copper zone on In3.Cu, net GND
Other:
- board text added: "+69420"
- board text added: "128MB HyperRAM!"
- board text added: "94V-0 E479892 JLC-1"
- board text added: "@mastodon.social"
- board text added: "@zeankun.dev"
- board text added: "C"
- board text added: "DESIGNED AND ASSEMBLED IN INDONESIA PCB MADE IN CHINA"
- board text added: "FIGHTER"
- board text added: "Lukas"
- board text added: "Nice disassembly by the way!"
- board text added: "RECOMMENDED BY:"
- board text added: "Regen/Damage"
- board text added: "TIP: check the back for lots of silkscreen artwork!"
- board text added: "Type-D HDMI out"
- board text added: "US"
- board text added: "USB-C"
- board text added: "Warranty Voided!"
- board text added: "Xilinx Spartan 6"
- board text added: "love it? i'd like to hear from you!"
- board text added: "this PCB is designed ASAP in NYE and zeankun.dev's 17th anniversary. happy bday!"
- board text added: "zeankun.dev's CastleBOX FPGA with Spartan 6"
- board text added: "zeankundev"
- board text added: "© 2025 zeankun.dev designed on 1/1/2025 (birthday)"
- board text added: "©️ 2025 zeankun.dev. logo ©️ choco panda kat all rights reserved"
