File: CastleBox/CastleBox.kicad_sch (KiCad schematic)
At the start: 43 parts, among them J1 USB_C_Receptacle_USB2.0_16P, J2 HDMI_C_1.4, J4 Conn_02x15_Odd_Even, U1 XC6SLX9-FTG256, U2 MIC5205YM5, U3 MIC5205YM5, U4 W955K8MBYA, U5 W955K8MBYA, U6 CY7C65215-32LTXI, X1 ASE-50MHz

Commit message: routine backup
Parts:
- added C19, C20: 0.1u, Capacitor_SMD:C_0402_1005Metric, symbol Device:C
- added R11, R12: 100k, Resistor_SMD:R_0402_1005Metric, symbol Device:R
- added U7: TXS0102YZP, Package_BGA:Texas_DSBGA-8_0.9x1.9mm_Layout2x4_P0.5mm, symbol Logic_LevelTranslator:TXS0102YZP
- J2: footprint Connector_Video:HDMI_Micro-D_Molex_46765-1x01 -> HDMI:VALCON_HD-RA-DSF12-TR
Connections:
- net +1V2: now also J4.2 (Pin_2)
- net +3V3: now also J4.27 (Pin_27), C19.2, U7.C1 (VCCA), U7.C2 (OE)
- net CK+: now also U1.B1 (IO_L50N_M3BA2_3)
- net CK-: now also U1.B2 (IO_L52P_M3A8_3)
- net D0+: now also U1.C1 (IO_L50P_M3WE_3)
- net D0-: now also U1.D1 (IO_L49N_M3A2_3)
- net D1+: now also U1.E1 (IO_L46N_M3CLKN_3)
- net D1-: now also U1.E2 (IO_L46P_M3CLK_3)
- net D2+: now also U1.G1 (IO_L40N_M3DQ7_3)
- net D2-: now also U1.F1 (IO_L41N_GCLK26_M3DQ5_3)
- net GND: now also J2.1 (D2S), J2.10 (CKS), J2.13 (GND), J2.4 (D1S), J2.7 (D0S), J2.SH, J4.22 (Pin_22), J4.30 (Pin_30), J4.4 (Pin_4), C19.1, C20.2, R11.1, U7.B1 (GND)
- net VBUS: now also J4.1 (Pin_1)
- net VSYS: now also J2.18 (+5V), J4.29 (Pin_29), C20.1, U7.B2 (VCCB)
- net PA4: now reaches J4.10 (Pin_10)
- net PA4: now also U1.A4 (IO_L1N_VREF_0)
- net PA6: now reaches J4.11 (Pin_11)
- net PA6: now also U1.A6 (IO_L4N_0)
- net PB5: now reaches J4.12 (Pin_12)
- net PB5: now also U1.B5 (IO_L2P_0)
- net PA7: now reaches J4.13 (Pin_13)
- net PA7: now also U1.A7 (IO_L6N_0)
- net PB6: now reaches J4.14 (Pin_14)
- net PB6: now also U1.B6 (IO_L4P_0)
- net PA8: now reaches J4.15 (Pin_15)
- net PA8: now also U1.A8 (IO_L33N_0)
- net PB8: now reaches J4.16 (Pin_16)
- net PB8: now also U1.B8 (IO_L33P_0)
- net PB10: now reaches J4.17 (Pin_17)
- net PB10: now also U1.B10 (IO_L35P_GCLK17_0)
- net PA9: now reaches J4.18 (Pin_18)
- net PA9: now also U1.A9 (IO_L34N_GCLK18_0)
- net PA11: now reaches J4.19 (Pin_19)
- net PA11: now also U1.A11 (IO_L39N_0)
- net PA12: now reaches J4.20 (Pin_20)
- net PA12: now also U1.A12 (IO_L62N_VREF_0)
- net PB12: now reaches J4.21 (Pin_21)
- net PB12: now also U1.B12 (IO_L62P_0)
- net PB14: now reaches J4.23 (Pin_23)
- net PB14: now also U1.B14 (IO_L65P_SCP3_0)
- net PA13: now reaches J4.24 (Pin_24)
- net PA13: now also U1.A13 (IO_L63N_SCP6_0)
- net PB15: now reaches J4.25 (Pin_25)
- net PB15: now also U1.B15 (IO_L29P_A23_M1A13_1)
- net PA14: now reaches J4.26 (Pin_26)
- net PA14: now also U1.A14 (IO_L65N_SCP2_0)
- net PA2: now reaches J4.3 (Pin_3)
- net PA2: now also U1.A2 (IO_L52N_M3A9_3)
- net PC3: now reaches J4.5 (Pin_5)
- net PC3: now also U1.C3 (IO_L48P_M3BA0_3)
- net PC2: now reaches J4.6 (Pin_6)
- net PC2: now also U1.C2 (IO_L48N_M3BA1_3)
- net PB3: now reaches J4.7 (Pin_7)
- net PB3: now also U1.B3 (IO_L83P_3)
- net PA3: now reaches J4.8 (Pin_8)
- net PA3: now also U1.A3 (IO_L83N_VREF_3)
- net PA5: now reaches J4.9 (Pin_9)
- net PA5: now also U1.A5 (IO_L2N_0)
- net DVI_SCL: now reaches U1.D3 (IO_L49P_M3A7_3)
- net DVI_SCL: now also U7.D2 (A1)
- net DVI_SDA: now reaches U1.E3 (IO_L54N_M3A11_3)
- net DVI_SDA: now also U7.D1 (A2)
- net DVI_HOTPLUG: now reaches U1.F2 (IO_L41P_GCLK27_M3DQ4_3)
- net DVI_HOTPLUG: now also R11.2, R12.1
- net at J2.15 (SCL): now also U7.A2 (B1)
- net at J2.16 (SDA): now also U7.A1 (B2)
- net at J2.19 (HPD/HEAC-): now also R12.2
- no-connect marks 18 -> 149
Other:
- moved on the sheet: J2
