File: LiPower-TP4056/LiPower-TP4056.kicad_pcb (KiCad board)
At the start: 2 copper layers, 18 x 25 mm, 26 parts, among them J1 USB_C_Receptacle_USB2.0, J2 Conn_01x02, J3 Conn_01x02, J4 Conn_01x02, Q1 FS8205A, U1 TP4056, U2 DW01A

Commit message: routine backup
Parts:
- moved G*** 1.10 mm to (93.1, 40.9)
