File: CastleBox_Pro/CastleBox_Pro.kicad_pcb (KiCad board)
At the start: 6 copper layers, 50 x 33 mm, 86 parts, among them J1 HDMI_C_1.4, J2 USB_C_Receptacle_USB2.0_16P, J3 Conn_02x15_Odd_Even, SW1 VSEL, U1 CY7C65215-32LTXI, U2 XC6SLX9-FTG256, U3 W955K8MBYA, U4 W955K8MBYA, U5 ATtiny406-M, U6 FUSB302B10MPX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

Commit message: fixed drc errors
Parts:
- moved C20 1.96 mm to (160.5, 54.0), turned to -90 degrees
Routing:
- net +3V3: track 46.5 -> 63.3 mm, vias 42 -> 32
- net +1V2: track 9.67 -> 11.9 mm, vias 16 -> 13
- net VBUS: track 51.2 -> 51.3 mm, vias 14 -> 13

Commit message: synced backup 6/3/2025
Parts:
- moved G*** 15.8 mm to (149.6, 65.2)
- moved G*** 0.69 mm to (143.9, 61.1)
- moved REF** 0.65 mm to (150.0, 56.5)
Routing:
- net VBUS: track 51.3 -> 62.5 mm, vias 13 -> 11
- net GND: track 57.9 -> 60.6 mm, vias 61 -> 63
Other:
- board text added: "Supports USB-C PD only on supported power bricks, such as JETE E11, UGREEN PD-compatible charger, or PPS chargers like the OEM Samsung 25W charger to charge your phone."
- board text added: "USB-C (65W) Power Delivery"
- board text added: "VSELCT"
- board text removed: "USB-C PD"
- board text removed: "Voltage Select"
- board text removed: "x2 PSRAM memory"

Commit message: sync to upstream 21/5/2025 06:52
Routing:
- net /D2-: track 19.0 -> 16.7 mm
