File: Deezplay-RP2350/Deezplay-RP2350.kicad_pcb (KiCad board)
At the start: 4 copper layers, 26 x 55 mm, 71 parts, among them J1 USB_C_Receptacle_USB2.0_16P, J2 Battery_Pad, J3 Conn_01x16, J4 Conn_01x16, Q1 BC807, SW1 SW_Push, SW2 SW_Push, U1 RP2350A, U2 ESP32-C3FN4, U3 W25Q32JVZP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

Commit message: sync to upstream 21/5/2025 06:52
Parts:
- moved C6 64.0 mm to (92.2, 71.1), turned to 90 degrees
- moved C11 22.2 mm to (90.6, 71.2), turned to 90 degrees
- moved C4 0.72 mm to (97.9, 75.8), turned to 0 degrees
- moved C9 0.46 mm to (94.9, 81.4)
Routing:
- net +1V1: track 0.00 -> 32.5 mm, vias 4 -> 7
- net Net-(U1-XOUT): track 13.6 -> 14.2 mm
