File: CastleBox_NeoPro/peripherals.kicad_sch (KiCad schematic)
At the start: 15 parts, among them J3 USB_A, J4 USB_A, J5 HDMI_A, U2 XC6SLX9-FTG256, U5 W955K8MBYA, U6 W955K8MBYA

Commit message: added SPI communication protocol
Connections:
- net FPGA_CS: now reaches U2.L13 (IO_L53N_VREF_1)
- net FPGA_MISO: now reaches U2.M13 (IO_L74P_AWAKE_1)
- net FPGA_MOSI: now reaches U2.M14 (IO_L74N_DOUT_BUSY_1)
- net FPGA_SCK: now reaches U2.R14 (IO_L50P_M1UDQS_1)
Changed lines of the file:
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@@
+	(wire
+		(pts
+			(xy 152.4 181.61) (xy 156.21 181.61)
+		)
+		(stroke
+			(width 0)
+			(type default)
+		)
+	)
 	(wire
 		(pts
@@
 	(wire
 		(pts
+			(xy 152.4 184.15) (xy 156.21 184.15)
+		)
+		(stroke
+			(width 0)
+			(type default)
+		)
+	)
+	(wire
+		(pts
 			(xy 231.14 90.17) (xy 231.14 88.9)
 		)
@@
 	(wire
 		(pts
+			(xy 152.4 161.29) (xy 156.21 161.29)
+		)
+		(stroke
+			(width 0)
+			(type default)
+		)
+	)
+	(wire
+		(pts
 			(xy 191.77 154.94) (xy 189.23 154.94)
 		)
@@
 		(pts
 			(xy 137.16 25.4) (xy 139.7 25.4)
+		)
+		(stroke
+			(width 0)
+			(type default)
+		)
+	)
+	(wire
+		(pts
+			(xy 152.4 179.07) (xy 156.21 179.07)
 		)
 		(stroke
@@
 		)
 	)
+	(global_label "FPGA_SCK"
+		(shape input)
+		(at 156.21 161.29 0)
+		(fields_autoplaced yes)
+		(effects
+			(font
+				(size 1.27 1.27)
+			)
+			(justify left)
+		)
+		(property "Intersheetrefs" "${INTERSHEET_REFS}"
+			(at 169.7822 161.29 0)
+			(effects
+				(font
+					(size 1.27 1.27)
+				)
+				(justify left)
+				(hide yes)
+			)
+		)
+	)
 	(global_label "HDMI_HPD"
 		(shape input)
@@
 				(hide yes)
 			)
+		)
+	)
+	(global_label "FPGA_MOSI"
+		(shape input)
+		(at 156.21 184.15 0)
+		(fields_autoplaced yes)
+		(effects
+			(font
+				(size 1.27 1.27)
+			)
+			(justify left)
+		)
+		(property "Intersheetrefs" "${INTERSHEET_REFS}"
+			(at 170.7128 184.15 0)
+			(effects
+				(font
+					(size 1.27 1.27)
+				)
+				(justify left)
+				(hide yes)
+			)
+		)
+	)
+	(global_label "FPGA_CS"
+		(shape input)
+		(at 156.21 179.07 0)
+		(fields_autoplaced yes)
+		(effects
+			(font
+				(size 1.27 1.27)
+			)
+			(justify left)
+		)
+		(property "Intersheetrefs" "${INTERSHEET_REFS}"
+			(at 168.4844 179.07 0)
+			(effects
+				(font
+					(size 1.27 1.27)
+				)
+				(justify left)
+				(hide yes)
+			)
+		)
+	)
+	(global_label "FPGA_MISO"
+		(shape input)
+		(at 156.21 181.61 0)
+		(fields_autoplaced yes)
+		(effects
+			(font
+				(size 1.27 1.27)
+			)
+			(justify left)
+		)
+		(property "Intersheetrefs" "${INTERSHEET_REFS}"
+			(at 170.7128 181.61 0)
+			(effects
+				(font
+					(size 1.27 1.27)
+				)
+				(justify left)
+				(hide yes)
+			)
