File: CastleBox_NeoPro/power.kicad_sch (KiCad schematic)
At the start: 0 parts

Commit message: added CastleBox NeoPro
Parts:
- added C1, C2, C3: 10u, Capacitor_SMD:C_0402_1005Metric, symbol Device:C
- added C10, C11, C12, C15: 4.7u, Capacitor_SMD:C_0402_1005Metric, symbol Device:C
- added C13, C16, C17: 0.47u, Capacitor_SMD:C_0402_1005Metric, symbol Device:C
- added C14, C9: 100u, Capacitor_SMD:C_0402_1005Metric, symbol Device:C
- added C4, C5: 10uF, Capacitor_SMD:C_0402_1005Metric, symbol Device:C
- added C7, C8: 0.1uF, Capacitor_SMD:C_0402_1005Metric, symbol Device:C
- added D1, D2: 1N5819HW-7-F, Diode_SMD:D_SOD-123, symbol Device:D
- added H1, H2, H3, H4: MountingHole, MountingHole:MountingHole_2.5mm, symbol Mechanical:MountingHole
- added J1: USB_RP2350A, Connector_USB:USB_C_Receptacle_GCT_USB4105-xx-A_16P_TopMnt_Horizontal, symbol Connector:USB_C_Receptacle_USB2.0_16P
- added J2: USB_FPGA, Connector_USB:USB_C_Receptacle_GCT_USB4105-xx-A_16P_TopMnt_Horizontal, symbol Connector:USB_C_Receptacle_USB2.0_16P
- added L1, L2: 2.2uH, Inductor_SMD:L_Changjiang_FNR252010S, symbol Device:L
- added R1, R2, R3, R4: 5.1k, Resistor_SMD:R_0402_1005Metric, symbol Device:R
- added R10, R13: 500k, Resistor_SMD:R_0402_1005Metric, symbol Device:R
- added R12: 680k, Resistor_SMD:R_0402_1005Metric, symbol Device:R
- added R5, R6, R7, R8: 27, Resistor_SMD:R_0402_1005Metric, symbol Device:R
- added R9: 150k, Resistor_SMD:R_0402_1005Metric, symbol Device:R
- added U1: EA3036, Package_DFN_QFN:WQFN-20-1EP_3x3mm_P0.4mm_EP1.7x1.7mm_ThermalVias, symbol Micro-SpecificLibs:EA3036
- added U2: XC6SLX9-FTG256, Package_BGA:BGA-256_17.0x17.0mm_Layout16x16_P1.0mm_Ball0.5mm_Pad0.4mm_NSMD, symbol FPGA_Xilinx_Spartan6:XC6SLX9-FTG256
Connections:
- new net: J2.A7 (D-), J2.B7 (D-), R7.1
- new net: J1.B5 (CC2), R2.1
- new net: R12.2, R9.2, U1.14 (FB1)
- new net: J2.B5 (CC2), R4.1
- new net: R10.2, R13.2, U1.3 (FB2)
- new net: J2.A6 (D+), J2.B6 (D+), R8.1
- new net: J2.A5 (CC1), R3.1
- new net: L1.2, U1.11 (SW1)
- new net: J1.A6 (D+), J1.B6 (D+), R6.1
- new net: J1.A7 (D-), J1.B7 (D-), R5.1
- new net: L2.2, U1.6 (SW2)
- new net: J1.A5 (CC1), R1.1
- new net +1V2: C10.1, C11.1, C12.1, C13.1, C5.1, C8.1, C9.1, L2.1, R13.1, U2.G7 (VCCINT), U2.G9 (VCCINT), U2.H10 (VCCINT), U2.H8 (VCCINT), U2.J7 (VCCINT), U2.J9 (VCCINT), U2.K10 (VCCINT), U2.K8 (VCCINT)
- new net +3V3: C14.1, C15.1, C16.1, C17.1, C4.1, C7.1, L1.1, R12.1, U2.E5 (VCCAUX), U2.F11 (VCCAUX), U2.F8 (VCCAUX), U2.G10 (VCCAUX), U2.H6 (VCCAUX), U2.J10 (VCCAUX), U2.L6 (VCCAUX), U2.L9 (VCCAUX)
- new net +5V: C1.1, C2.1, C3.1, D1.1 (K), D2.1 (K), U1.10 (VIN1), U1.16 (VCC), U1.18 (EN3), U1.19 (VIN3), U1.7 (VIN2), U1.8 (EN2), U1.9 (EN1)
- new net FTDI_D+: R8.2
- new net FTDI_D-: R7.2
- new net GND: C1.2, C10.2, C11.2, C12.2, C13.2, C14.2, C15.2, C16.2, C17.2, C2.2, C3.2, C4.2, C5.2, C7.2, C8.2, C9.2, J1.A1 (GND), J1.A12 (GND), J1.B1 (GND), J1.B12 (GND), J1.S1 (SHIELD), J2.A1 (GND), J2.A12 (GND), J2.B1 (GND), J2.B12 (GND), J2.S1 (SHIELD), R1.2, R10.1, R2.2, R3.2, R4.2, R9.1, U1.1 (GND), U1.12 (GND), U1.13 (AGND), U1.15 (AGND), U1.17 (AGND), U1.21 (EPAD), U1.4 (AGND), U1.5 (GND), U2.A1 (GND), U2.A16 (GND), U2.B11 (GND), U2.B7 (GND), U2.D13 (GND), U2.D4 (GND), U2.E9 (GND), U2.G15 (GND), U2.G2 (GND), U2.G8 (GND), U2.H12 (GND), U2.H7 (GND), U2.H9 (GND), U2.J5 (GND), U2.J8 (GND), U2.K7 (GND), U2.K9 (GND), U2.L15 (GND), U2.L2 (GND), U2.M8 (GND), U2.N13 (GND), U2.P3 (GND), U2.R10 (GND), U2.R6 (GND), U2.T1 (GND), U2.T16 (GND)
- new net MCU_D+: R6.2
- new net MCU_D-: R5.2
- new net VBUSA: D1.2 (A), J1.A4 (VBUS), J1.A9 (VBUS), J1.B4 (VBUS), J1.B9 (VBUS)
- new net VBUSB: D2.2 (A), J2.A4 (VBUS), J2.A9 (VBUS), J2.B4 (VBUS), J2.B9 (VBUS)
- no-connect marks 0 -> 6
